Commit message: fix(urdf)!: align zedxm.xacro with official zed-ros2-wrapper geometry
BREAKING CHANGE: Frame names renamed from zedx_* to zedxm_* to match
camera model. Left camera Y offset sign corrected from -baseline_half
to +baseline_half per ROS convention.

- Fix left camera Y offset: -baseline_half → +baseline_half (left = +Y)
- Rename all frame prefixes: zedx_ → zedxm_ (match ZED X Mini model)
- Add optical_offset_x (-0.01m) to left/right eye joints
- Add right camera frame (zedxm_right_optical_frame) and depth optical
- Add IMU link (zedxm_imu_link) with Camera-IMU offset from ZED SDK
- Bump version to 0.2.0 with migration guide in CHANGELOG

Co-Authored-By: Claude Opus 4.6 (1M context) <noreply@anthropic.com>

File: urdf/zedxm.xacro (robot description, xacro)
@@ -11,8 +11,14 @@
         <!-- Half-baseline: left/right eye offset from camera body center -->
         <xacro:property name="baseline_half" value="0.025"/>
+        <!-- Optical center offset from body center (lens 10mm behind body center) -->
+        <!-- Value from zed-ros2-wrapper zed_macro.urdf.xacro for ZED X Mini -->
+        <xacro:property name="optical_offset_x" value="-0.01"/>
+        <!-- IMU offset from body center (Camera-IMU Translation from ZED SDK calibration) -->
+        <xacro:property name="imu_offset_y" value="-0.034502"/>
+        <xacro:property name="imu_offset_z" value="-0.004356"/>
         <!-- Camera housing link -->
-        <!-- zedx_link frame = camera body center (mount reference point) -->
+        <!-- zedxm_link frame = camera body center (mount reference point) -->
         <!-- Collision: conservative box around housing -->
-        <link name="${prefix}zedx_link">
+        <link name="${prefix}zedxm_link">
             <inertial>
                 <origin xyz="0 0 -0.030" rpy="0 0 0"/>
@@ -22,9 +28,10 @@
             </inertial>
             <visual>
+                <!-- STL exported in non-ROS axes; rpy corrects to x-forward, y-left, z-up -->
                 <origin xyz="0 0 -0.016" rpy="${radians(-90)} ${radians(-90)} ${radians(-90)}"/>
                 <geometry>
                     <mesh filename="package://stereolabs_description/meshes/zedxm/zedxm.stl"/>
                 </geometry>
-                <material name="zedx_dark">
+                <material name="zedxm_dark">
                     <color rgba="0.25 0.25 0.25 1.0"/>
                 </material>
@@ -38,26 +45,50 @@
         </link>
         <!-- Left eye optical center (hand-eye calibration reference, depth origin) -->
-        <link name="${prefix}zedx_left_optical_frame"/>
-        <!-- Depth optical frame (ROS convention: z-forward, x-right, y-down) -->
-        <link name="${prefix}zedx_depth_optical_frame"/>
+        <link name="${prefix}zedxm_left_optical_frame"/>
+        <!-- Left depth optical frame (ROS convention: z-forward, x-right, y-down) -->
+        <link name="${prefix}zedxm_depth_optical_frame"/>
+        <!-- Right eye optical center -->
+        <link name="${prefix}zedxm_right_optical_frame"/>
+        <!-- Right depth optical frame (ROS convention: z-forward, x-right, y-down) -->
+        <link name="${prefix}zedxm_right_depth_optical_frame"/>
+        <!-- IMU link -->
+        <link name="${prefix}zedxm_imu_link"/>
         <!-- Mount joint: parent_link -> camera body center -->
         <!-- Transform from Hand-Eye calibration YAML -->
-        <joint name="${prefix}zedx_mount_joint" type="fixed">
+        <joint name="${prefix}zedxm_mount_joint" type="fixed">
             <origin xyz="${cam_mount['x']} ${cam_mount['y']} ${cam_mount['z']}"
                     rpy="${cam_mount['roll']} ${cam_mount['pitch']} ${cam_mount['yaw']}"/>
             <parent link="${parent_link}"/>
-            <child link="${prefix}zedx_link"/>
+            <child link="${prefix}zedxm_link"/>
         </joint>
-        <!-- Camera body center -> left eye (-baseline/2 in y) -->
-        <joint name="${prefix}zedx_left_eye_joint" type="fixed">
-            <origin xyz="0 -${baseline_half} 0" rpy="0 0 0"/>
-            <parent link="${prefix}zedx_link"/>
-            <child link="${prefix}zedx_left_optical_frame"/>
+        <!-- Camera body center -> left eye (+baseline/2 in y, ROS convention: left = +Y) -->
+        <joint name="${prefix}zedxm_left_eye_joint" type="fixed">
+            <origin xyz="${optical_offset_x} ${baseline_half} 0" rpy="0 0 0"/>
+            <parent link="${prefix}zedxm_link"/>
+            <child link="${prefix}zedxm_left_optical_frame"/>
         </joint>
         <!-- Left eye -> depth optical frame (camera body -> ROS optical axes) -->
-        <joint name="${prefix}zedx_optical_joint" type="fixed">
+        <joint name="${prefix}zedxm_optical_joint" type="fixed">
             <origin xyz="0 0 0" rpy="${radians(-90)} 0 ${radians(-90)}"/>
-            <parent link="${prefix}zedx_left_optical_frame"/>
-            <child link="${prefix}zedx_depth_optical_frame"/>
+            <parent link="${prefix}zedxm_left_optical_frame"/>
+            <child link="${prefix}zedxm_depth_optical_frame"/>
+        </joint>
+        <!-- Camera body center -> right eye (-baseline/2 in y) -->
+        <joint name="${prefix}zedxm_right_eye_joint" type="fixed">
+            <origin xyz="${optical_offset_x} -${baseline_half} 0" rpy="0 0 0"/>
+            <parent link="${prefix}zedxm_link"/>
+            <child link="${prefix}zedxm_right_optical_frame"/>
+        </joint>
+        <!-- Right eye -> depth optical frame (camera body -> ROS optical axes) -->
+        <joint name="${prefix}zedxm_right_optical_joint" type="fixed">
+            <origin xyz="0 0 0" rpy="${radians(-90)} 0 ${radians(-90)}"/>
+            <parent link="${prefix}zedxm_right_optical_frame"/>
+            <child link="${prefix}zedxm_right_depth_optical_frame"/>
+        </joint>
+        <!-- Camera body center -> IMU -->
+        <joint name="${prefix}zedxm_imu_joint" type="fixed">
+            <origin xyz="0 ${imu_offset_y} ${imu_offset_z}" rpy="0 0 0"/>
+            <parent link="${prefix}zedxm_link"/>
+            <child link="${prefix}zedxm_imu_link"/>
         </joint>
     </xacro:macro>

Commit message: fix(urdf)!: revert eye offset signs and remove optical_offset_x for plem body frame
plem body frame은 mesh rpy(-90,-90,-90) 보정으로 공식 zed-ros2-wrapper와
축 방향이 다르다. v0.2.0의 baseline 부호 변경과 optical_offset_x 적용이
RViz 검증에서 물리적 현실과 불일치 확인되어 원복한다.

- left eye Y: +baseline_half → -baseline_half (plem: left = -Y)
- right eye Y: -baseline_half → +baseline_half
- optical_offset_x 제거 (plem body frame에서 적용 불가)
- Bump version to 0.2.1

Co-Authored-By: Claude Opus 4.6 (1M context) <noreply@anthropic.com>

File: urdf/zedxm.xacro (robot description, xacro)
@@ -11,7 +11,8 @@
         <!-- Half-baseline: left/right eye offset from camera body center -->
         <xacro:property name="baseline_half" value="0.025"/>
-        <!-- Optical center offset from body center (lens 10mm behind body center) -->
-        <!-- Value from zed-ros2-wrapper zed_macro.urdf.xacro for ZED X Mini -->
-        <xacro:property name="optical_offset_x" value="-0.01"/>
+        <!-- optical_offset_x not applied: plem body frame axes differ from
+             official zed-ros2-wrapper (mesh rpy(-90,-90,-90) correction),
+             so the official X offset value does not transfer directly.
+             Pre-v0.2.0 URDF operated correctly without it. -->
         <!-- IMU offset from body center (Camera-IMU Translation from ZED SDK calibration) -->
         <xacro:property name="imu_offset_y" value="-0.034502"/>
@@ -62,7 +63,7 @@
             <child link="${prefix}zedxm_link"/>
         </joint>
-        <!-- Camera body center -> left eye (+baseline/2 in y, ROS convention: left = +Y) -->
+        <!-- Camera body center -> left eye (-baseline/2 in y, plem body frame: left = -Y) -->
         <joint name="${prefix}zedxm_left_eye_joint" type="fixed">
-            <origin xyz="${optical_offset_x} ${baseline_half} 0" rpy="0 0 0"/>
+            <origin xyz="0 -${baseline_half} 0" rpy="0 0 0"/>
             <parent link="${prefix}zedxm_link"/>
             <child link="${prefix}zedxm_left_optical_frame"/>
@@ -74,7 +75,7 @@
             <child link="${prefix}zedxm_depth_optical_frame"/>
         </joint>
-        <!-- Camera body center -> right eye (-baseline/2 in y) -->
+        <!-- Camera body center -> right eye (+baseline/2 in y, plem body frame: right = +Y) -->
         <joint name="${prefix}zedxm_right_eye_joint" type="fixed">
-            <origin xyz="${optical_offset_x} -${baseline_half} 0" rpy="0 0 0"/>
+            <origin xyz="0 ${baseline_half} 0" rpy="0 0 0"/>
             <parent link="${prefix}zedxm_link"/>
             <child link="${prefix}zedxm_right_optical_frame"/>
